File: business_card.kicad_sch (KiCad schematic)
At the start: 66 parts, among them J1 USB_C_Receptacle_USB2.0_14P, J10 CAP_TOUCH_RECT, J11 CAP_TOUCH_RECT, J12 CAP_TOUCH_RECT, J13 CAP_TOUCH_CIRC, J2 CAP_TOUCH_CIRC, J3 CAP_TOUCH_RECT, J4 CAP_TOUCH_RECT, J5 CAP_TOUCH_RECT, J6 CAP_TOUCH_RECT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

Commit message: increase ic distance to .22mm
Parts:
- C1, C17, C2, C20, C3, C4, C5, C6: Distributor Link https://www.digikey.com/en/products/detail/murata-electronics/GRM0335C1E100JA01D/4358173 -> https://www.digikey.com/en/products/detail/murata-electronics/GRM033C71C104KE14D/5027472; MPN GRM0335C1E100JA01D -> GRM033C71C104KE14D
- Y1: Distributor Link https://www.digikey.com/en/products/detail/nextgen-componen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 -> https://www.digikey.com/en/products/detail/ndk-nihon-dempa-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; MPN XV32M00000S409 -> END4263D-32M; Manufacturer TGS -> NDK (NIHON DEMPA KOGYO CO., LTD)
Changed lines of the file:
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@@
 			)
 		)
-		(property "Distributor Link" "https://www.digikey.com/en/products/detail/murata-electronics/GRM0335C1E100JA01D/4358173"
+		(property "Distributor Link" "https://www.digikey.com/en/products/detail/murata-electronics/GRM033C71C104KE14D/5027472"
 			(at 175.26 24.13 0)
 			(effects
@@
 			)
 		)
-		(property "MPN" "GRM0335C1E100JA01D"
+		(property "MPN" "GRM033C71C104KE14D"
 			(at 175.26 24.13 0)
 			(effects
@@
 			)
 		)
-		(property "Distributor Link" "https://www.digikey.com/en/products/detail/murata-electronics/GRM0335C1E100JA01D/4358173"
+		(property "Distributor Link" "https://www.digikey.com/en/products/detail/murata-electronics/GRM033C71C104KE14D/5027472"
 			(at 210.82 24.13 0)
 			(effects
@@
 			)
 		)
-		(property "MPN" "GRM0335C1E100JA01D"
+		(property "MPN" "GRM033C71C104KE14D"
 			(at 210.82 24.13 0)
 			(effects
@@
 			)
 		)
-		(property "Distributor Link" "https://www.digikey.com/en/products/detail/murata-electronics/GRM0335C1E100JA01D/4358173"
+		(property "Distributor Link" "https://www.digikey.com/en/products/detail/murata-electronics/GRM033C71C104KE14D/5027472"
 			(at 201.93 24.13 0)
 			(effects
@@
 			)
 		)
-		(property "MPN" "GRM0335C1E100JA01D"
+		(property "MPN" "GRM033C71C104KE14D"
 			(at 201.93 24.13 0)
 			(effects
@@
 			)
 		)
-		(property "Distributor Link" "https://www.digikey.com/en/products/detail/murata-electronics/GRM0335C1E100JA01D/4358173"
+		(property "Distributor Link" "https://www.digikey.com/en/products/detail/murata-electronics/GRM033C71C104KE14D/5027472"
 			(at 138.43 24.13 0)
 			(effects
@@
 			)
 		)
-		(property "MPN" "GRM0335C1E100JA01D"
+		(property "MPN" "GRM033C71C104KE14D"
 			(at 138.43 24.13 0)
 			(effects
@@
 			)
 		)
-		(property "Distributor Link" "https://www.digikey.com/en/products/detail/murata-electronics/GRM0335C1E100JA01D/4358173"
+		(property "Distributor Link" "https://www.digikey.com/en/products/detail/murata-electronics/GRM033C71C104KE14D/5027472"
 			(at 124.46 172.72 90)
 			(effects
@@
 			)
 		)
-		(property "MPN" "GRM0335C1E100JA01D"
+		(property "MPN" "GRM033C71C104KE14D"
 			(at 124.46 172.72 90)
 			(effects
@@
 			)
 		)
-		(property "Distributor Link" "https://www.digikey.com/en/products/detail/murata-electronics/GRM0335C1E100JA01D/4358173"
+		(property "Distributor Link" "https://www.digikey.com/en/products/detail/murata-electronics/GRM033C71C104KE14D/5027472"
 			(at 184.15 24.13 0)
 			(effects
@@
 			)
 		)
-		(property "MPN" "GRM0335C1E100JA01D"
+		(property "MPN" "GRM033C71C104KE14D"
 			(at 184.15 24.13 0)
 			(effects
@@
 			)
 		)
-		(property "Distributor Link" "https://www.digikey.com/en/products/detail/murata-electronics/GRM0335C1E100JA01D/4358173"
+		(property "Distributor Link" "https://www.digikey.com/en/products/detail/murata-electronics/GRM033C71C104KE14D/5027472"
 			(at 193.04 24.13 0)
 			(effects
@@
 			)
 		)
-		(property "MPN" "GRM0335C1E100JA01D"
+		(property "MPN" "GRM033C71C104KE14D"
 			(at 193.04 24.13 0)
 			(effects
@@
 			)
 		)
-		(property "Datasheet" "https://mm.digikey.com/Volume0/opasdata/d220001/medias/docus/4831/XV32M00000S409.pdf"
+		(property "Datasheet" "https://mm.digikey.com/Volume0/opasdata/d220001/medias/docus/6257/ETS11B-07494.pdf"
 			(at 121.92 129.54 0)
 			(effects
@@
 			)
 		)
-		(property "Distributor Link" "https://www.digikey.com/en/products/detail/nextgen-components/XV32M00000S409/17942242?s=N4IgTCBcDaIBoDUDMYCyAGTmDKAWdAnCALoC%2BQA"
+		(property "Distributor Link" "https://www.digikey.com/en/products/detail/ndk-nihon-dempa-kogyo-co-ltd/END4263D-32M/24390080"
 			(at 121.92 129.54 0)
 			(effects
@@
 			)
 		)
-		(property "Manufacturer" "TGS"
+		(property "Manufacturer" "NDK (NIHON DEMPA KOGYO CO., LTD)"
 			(at 121.92 129.54 0)
 			(effects
@@
 			)
 		)
-		(property "MPN" "XV32M00000S409"
+		(property "MPN" "END4263D-32M"
 			(at 121.92 129.54 0)
 			(effects
@@
 			)
 		)
-		(property "Distributor Link" "https://www.digikey.com/en/products/detail/murata-electronics/GRM0335C1E100JA01D/4358173"
+		(property "Distributor Link" "https://www.digikey.com/en/products/detail/murata-electronics/GRM033C71C104KE14D/5027472"
 			(at 124.46 181.61 0)
 			(effects
@@
 			)
 		)
-		(property "MPN" "GRM0335C1E100JA01D"
+		(property "MPN" "GRM033C71C104KE14D"
 			(at 124.46 181.61 0)
 			(effects
